Commit message: Reward filed, but not working :'(

File: assets/gate.urdf (robot description, URDF)
Before this commit: robot test.urdf, 5 links, 4 joints
Links:
- link arrow: mass None -> 10
- link bottomBar: mass None -> 10
- link leftBar: mass None -> 10
- link rightBar: mass None -> 10
- link topBar: mass None -> 10
